Commit message: changee

File: src/kjk_urdf/urdf/kjk_urdf.urdf (robot description, URDF)
Before this commit: robot kjk, 3 links, 2 joints
Links:
- removed link wheel1_link
- removed link wheel2_link
- added link front_left_wheel_link; visual cylinder length=0.2 radius=0.2
- added link front_right_wheel_link; visual cylinder length=0.2 radius=0.2
- added link rear_left_wheel_link; visual cylinder length=0.2 radius=0.2
- added link rear_right_wheel_link; visual cylinder length=0.2 radius=0.2
- link body_link: geometry visual box size=2 10 0.5
Joints:
- removed joint wheel1_joint
- removed joint wheel2_joint
- added joint front_left_wheel_joint: type continuous, parent body_link, child front_left_wheel_link, origin xyz=0.9 -0.5 0 rpy=0 0 0, axis 0 1 0
- added joint front_right_wheel_joint: type continuous, parent body_link, child front_right_wheel_link, origin xyz=0.9 0.5 0 rpy=0 0 0, axis 0 1 0
- added joint rear_left_wheel_joint: type continuous, parent body_link, child rear_left_wheel_link, origin xyz=-0.9 -0.5 0 rpy=0 0 0, axis 0 1 0
- added joint rear_right_wheel_joint: type continuous, parent body_link, child rear_right_wheel_link, origin xyz=-0.9 0.5 0 rpy=0 0 0, axis 0 1 0

Commit message: motoreeeee

File: src/kjk_urdf/urdf/kjk_urdf.urdf (robot description, URDF)
Before this commit: robot kjk_car, 5 links, 4 joints
Links:
- link body_link: geometry visual box size=2 1 0.5
